File: Board.sch (EAGLE design)
At the start: 5 parts, among them U1 ATMEGA2560-16AU, U2 DRV8825PWPR, U3 DRV8825PWPR, U4 DRV8825PWPR, U5 LMZ22005TZ

Commit message: Added changes
Parts:
- removed U2, U3, U4: DRV8825PWPR, cartesian_main:DRV8825PWPR
- added J$1: USB-B1HSW6, cartesian_main:USB-B1HSW6
- added U6, U7, U8: DRV8825PWPR, cartesian_main:DRV8825PWPR
Changed lines of the file:
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@@
 <parts>
 <part name="U1" library="cartesian_main" deviceset="ATMEGA2560-16AU" device=""/>
-<part name="U2" library="cartesian_main" deviceset="DRV8825PWPR" device=""/>
-<part name="U3" library="cartesian_main" deviceset="DRV8825PWPR" device=""/>
-<part name="U4" library="cartesian_main" deviceset="DRV8825PWPR" device=""/>
 <part name="U5" library="cartesian_main" deviceset="LMZ22005TZ" device=""/>
+<part name="J$1" library="cartesian_main" deviceset="USB-B1HSW6" device=""/>
+<part name="U6" library="cartesian_main" deviceset="DRV8825PWPR" device=""/>
+<part name="U7" library="cartesian_main" deviceset="DRV8825PWPR" device=""/>
+<part name="U8" library="cartesian_main" deviceset="DRV8825PWPR" device=""/>
 </parts>
 <sheets>
 <sheet>
+<description>Control</description>
 <plain>
 </plain>
@@
 <attribute name="VALUE" x="-5.287190625" y="-88.0013" size="2.08436875" layer="96" ratio="10" rot="SR0"/>
 </instance>
-<instance part="U2" gate="G$1" x="502.92" y="124.46" smashed="yes">
-<attribute name="NAME" x="487.632" y="172.8717" size="1.783590625" layer="95"/>
-<attribute name="VALUE" x="487.6492" y="71.0121" size="1.7816" layer="96"/>
-</instance>
-<instance part="U3" gate="G$1" x="502.92" y="7.62" smashed="yes">
-<attribute name="NAME" x="487.632" y="56.0317" size="1.783590625" layer="95"/>
-<attribute name="VALUE" x="487.6492" y="-45.8279" size="1.7816" layer="96"/>
-</instance>
-<instance part="U4" gate="G$1" x="502.92" y="-101.6" smashed="yes">
-<attribute name="NAME" x="487.632" y="-53.1883" size="1.783590625" layer="95"/>
-<attribute name="VALUE" x="487.6492" y="-155.0479" size="1.7816" layer="96"/>
+<instance part="J$1" gate="G$1" x="-35.56" y="101.6" smashed="yes">
+<attribute name="NAME" x="-35.56" y="122.682" size="1.778" layer="95"/>
+<attribute name="VALUE" x="-35.56" y="99.06" size="1.778" layer="96"/>
 </instance>
 </instances>
@@
 </sheet>
 <sheet>
+<description>Power</description>
 <plain>
 </plain>
@@
 </instance>
 </instances>
+<busses>
+</busses>
+<nets>
+</nets>
+</sheet>
+<sheet>
+<description>Stepper Motor Drivers</description>
+<plain>
+</plain>
+<instances>
+<instance part="U6" gate="G$1" x="0" y="114.3" smashed="yes">
+<attribute name="NAME" x="-15.288" y="162.7117" size="1.783590625" layer="95"/>
+<attribute name="VALUE" x="-15.2708" y="60.8521" size="1.7816" layer="96"/>
+</instance>
+<instance part="U7" gate="G$1" x="0" y="-2.54" smashed="yes">
+<attribute name="NAME" x="-15.288" y="45.8717" size="1.783590625" layer="95"/>
+<attribute name="VALUE" x="-15.2708" y="-55.9879" size="1.7816" layer="96"/>
+</instance>
+<instance part="U8" gate="G$1" x="0" y="-111.76" smashed="yes">
+<attribute name="NAME" x="-15.288" y="-63.3483" size="1.783590625" layer="95"/>
+<attribute name="VALUE" x="-15.2708" y="-165.2079" size="1.7816" layer="96"/>
+</instance>
+</instances>

Commit message: Added more parts
Parts:
- added J$2: USB-B1HSW6, cartesian_main:USB-B1HSW6
- added U$1: WE_649004113322, cartesian_main:WE_649004113322
Other:
- note added: "5V REG"
- note added: "POWER SWITCH"
Changed lines of the file:
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@@
 <part name="U7" library="cartesian_main" deviceset="DRV8825PWPR" device=""/>
 <part name="U8" library="cartesian_main" deviceset="DRV8825PWPR" device=""/>
+<part name="J$2" library="cartesian_main" deviceset="USB-B1HSW6" device=""/>
+<part name="U$1" library="cartesian_main" deviceset="WE_649004113322" device=""/>
 </parts>
 <sheets>
@@
 <description>Power</description>
 <plain>
+<text x="-96.52" y="43.18" size="1.778" layer="91">POWER SWITCH</text>
+<text x="-91.44" y="5.08" size="1.778" layer="91">5V REG</text>
 </plain>
 <instances>
-<instance part="U5" gate="G$1" x="0" y="0" smashed="yes">
-<attribute name="VALUE" x="-15.2516" y="-13.3451" size="2.5487" layer="96"/>
-<attribute name="NAME" x="-15.2691" y="13.3605" size="2.553109375" layer="95"/>
+<instance part="U5" gate="G$1" x="-86.36" y="-12.7" smashed="yes">
+<attribute name="VALUE" x="-101.6116" y="-26.0451" size="2.5487" layer="96"/>
+<attribute name="NAME" x="-101.6291" y="0.6605" size="2.553109375" layer="95"/>
+</instance>
+<instance part="U$1" gate="G$1" x="-81.28" y="27.94" smashed="yes">
+<attribute name="NAME" x="-91.44" y="38.608" size="1.778" layer="95"/>
+<attribute name="VALUE" x="-91.44" y="22.86" size="1.778" layer="96"/>
 </instance>
 </instances>
@@
 </instance>
 </instances>
+<busses>
+</busses>
+<nets>
+</nets>
+</sheet>
+<sheet>
+<description>Tool Passthrough</description>
+<plain>
+</plain>
+<instances>
+<instance part="J$2" gate="G$1" x="0" y="0" smashed="yes">
+<attribute name="NAME" x="0" y="21.082" size="1.778" layer="95"/>
+<attribute name="VALUE" x="0" y="-2.54" size="1.778" layer="96"/>
+</instance>
+</instances>

Commit message: Adding more components
Parts:
- added U$2, U$3, U$4: 4P_MOLEX_KK254, cartesian_main:4P_MOLEX_KK254
- added U$5, U$6: ICSP_HDR, cartesian_main:ICSP_HDR
- added U$7: WE_649004113322, cartesian_main:WE_649004113322
- added U2: ATMEGA8U2-MU, cartesian_main:ATMEGA8U2-MU
Connections:
- new net 0: U$5.GND, U$6.GND, U$7.P$4, U1.GND, U1.GND_2, U1.GND_3, U1.GND_4, U1.GND_5
- new net 12V: U$7.P$2
- new net 24V: U$7.P$1
- new net 5V: U$7.P$3
- new net N$3: J$1.SHIELD, J$1.SHIELD2
Other:
- note added: "POWER OUTPUT"
- moved on the sheet: J$1
Changed lines of the file:
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@@
 <layer number="97" name="Info" color="7" fill="1" visible="yes" active="yes"/>
 <layer number="98" name="Guide" color="6" fill="1" visible="yes" active="yes"/>
+<layer number="99" name="SpiceOrder" color="7" fill="1" visible="yes" active="yes"/>
 </layers>
 <schematic xreflabel="%F%N/%S.%C%R" xrefpart="/%S.%C%R">
@@
 <part name="J$2" library="cartesian_main" deviceset="USB-B1HSW6" device=""/>
 <part name="U$1" library="cartesian_main" deviceset="WE_649004113322" device=""/>
+<part name="U$2" library="cartesian_main" deviceset="4P_MOLEX_KK254" device=""/>
+<part name="U$3" library="cartesian_main" deviceset="4P_MOLEX_KK254" device=""/>
+<part name="U$4" library="cartesian_main" deviceset="4P_MOLEX_KK254" device=""/>
+<part name="U2" library="cartesian_main" deviceset="ATMEGA8U2-MU" device=""/>
+<part name="U$5" library="cartesian_main" deviceset="ICSP_HDR" device=""/>
+<part name="U$6" library="cartesian_main" deviceset="ICSP_HDR" device=""/>
+<part name="U$7" library="cartesian_main" deviceset="WE_649004113322" device=""/>
+<part name="X_1" library="ngspice-simulation" library_urn="urn:adsk.eagle:library:527439" deviceset="GND" device=""/>
+<part name="X_2" library="ngspice-simulation" library_urn="urn:adsk.eagle:library:527439" deviceset="GND" device=""/>
+<part name="X_3" library="ngspice-simulation" library_urn="urn:adsk.eagle:library:527439" deviceset="GND" device=""/>
+<part name="X_4" library="ngspice-simulation" library_urn="urn:adsk.eagle:library:527439" deviceset="GND" device=""/>
 </parts>
 <sheets>
@@
 <instances>
 <instance part="U1" gate="A" x="0" y="0" smashed="yes">
-<attribute name="NAME" x="-6.050809375" y="80.9995" size="2.08473125" layer="95" ratio="10" rot="SR0"/>
-<attribute name="VALUE" x="-5.287190625" y="-88.0013" size="2.08436875" layer="96" ratio="10" rot="SR0"/>
-</instance>
-<instance part="J$1" gate="G$1" x="-35.56" y="101.6" smashed="yes">
-<attribute name="NAME" x="-35.56" y="122.682" size="1.778" layer="95"/>
-<attribute name="VALUE" x="-35.56" y="99.06" size="1.778" layer="96"/>
-</instance>
-</instances>
-<busses>
-</busses>
-<nets>
+<attribute name="NAME" x="-40.594809375" y="79.4755" size="2.08473125" layer="95" ratio="10" rot="SR0"/>
+<attribute name="VALUE" x="-41.101190625" y="-86.4773" size="2.08436875" layer="96" ratio="10" rot="SR0"/>
+</instance>
+<instance part="J$1" gate="G$1" x="-139.7" y="2.54" smashed="yes" rot="MR0">
+<attribute name="NAME" x="-139.7" y="23.622" size="1.778" layer="95" rot="MR0"/>
+<attribute name="VALUE" x="-139.7" y="0" size="1.778" layer="96" rot="MR0"/>
+</instance>
+<instance part="U2" gate="A" x="241.3" y="15.24" smashed="yes">
+<attribute name="NAME" x="220.18458125" y="44.3373" size="2.08565" layer="95" ratio="10" rot="SR0"/>
+<attribute name="VALUE" x="219.60295" y="-23.6253" size="2.0857" layer="96" ratio="10" rot="SR0"/>
+</instance>
+<instance part="U$5" gate="G$1" x="-96.52" y="96.52" smashed="yes"/>
+<instance part="U$6" gate="G$1" x="185.42" y="96.52" smashed="yes"/>
+<instance part="X_2" gate="G$1" x="210.82" y="96.52" smashed="yes"/>
+<instance part="X_3" gate="G$1" x="-71.12" y="96.52" smashed="yes"/>
+<instance part="X_4" gate="G$1" x="-50.8" y="-83.82" smashed="yes"/>
+</instances>
+<busses>
+</busses>
+<nets>
+<net name="0" class="0">
+<segment>
+<pinref part="U$6" gate="G$1" pin="GND"/>
+<wire x1="208.28" y1="99.06" x2="210.82" y2="99.06" width="0.1524" layer="91"/>
+<wire x1="210.82" y1="99.06" x2="210.82" y2="96.52" width="0.1524" layer="91"/>
+<pinref part="X_2" gate="G$1" pin="0"/>
+</segment>
+<segment>
+<pinref part="U$5" gate="G$1" pin="GND"/>
+<wire x1="-73.66" y1="99.06" x2="-71.12" y2="99.06" width="0.1524" layer="91"/>
+<wire x1="-71.12" y1="99.06" x2="-71.12" y2="96.52" width="0.1524" layer="91"/>
+<pinref part="X_3" gate="G$1" pin="0"/>
+</segment>
+<segment>
+<pinref part="U1" gate="A" pin="GND_2"/>
+<wire x1="-45.72" y1="-68.58" x2="-50.8" y2="-68.58" width="0.1524" layer="91"/>
+<wire x1="-50.8" y1="-68.58" x2="-50.8" y2="-71.12" width="0.1524" layer="91"/>
+<pinref part="U1" gate="A" pin="GND"/>
+<wire x1="-50.8" y1="-71.12" x2="-50.8" y2="-73.66" width="0.1524" layer="91"/>
+<wire x1="-50.8" y1="-73.66" x2="-50.8" y2="-76.2" width="0.1524" layer="91"/>
+<wire x1="-50.8" y1="-76.2" x2="-50.8" y2="-78.74" width="0.1524" layer="91"/>
+<wire x1="-50.8" y1="-78.74" x2="-50.8" y2="-83.82" width="0.1524" layer="91"/>
+<wire x1="-45.72" y1="-78.74" x2="-50.8" y2="-78.74" width="0.1524" layer="91"/>
+<junction x="-50.8" y="-78.74"/>
+<pinref part="U1" gate="A" pin="GND_5"/>
+<wire x1="-45.72" y1="-76.2" x2="-50.8" y2="-76.2" width="0.1524" layer="91"/>
+<junction x="-50.8" y="-76.2"/>
+<pinref part="U1" gate="A" pin="GND_4"/>
+<wire x1="-45.72" y1="-73.66" x2="-50.8" y2="-73.66" width="0.1524" layer="91"/>
+<junction x="-50.8" y="-73.66"/>
+<pinref part="U1" gate="A" pin="GND_3"/>
+<wire x1="-45.72" y1="-71.12" x2="-50.8" y2="-71.12" width="0.1524" layer="91"/>
+<junction x="-50.8" y="-71.12"/>
+<pinref part="X_4" gate="G$1" pin="0"/>
+</segment>
+</net>
+<net name="N$3" class="0">
+<segment>
+<pinref part="J$1" gate="G$1" pin="SHIELD2"/>
+<wire x1="-134.62" y1="7.62" x2="-129.54" y2="7.62" width="0.1524" layer="91"/>
+<pinref part="J$1" gate="G$1" pin="SHIELD"/>
+<wire x1="-129.54" y1="7.62" x2="-129.54" y2="5.08" width="0.1524" layer="91"/>
+<wire x1="-129.54" y1="5.08" x2="-134.62" y2="5.08" width="0.1524" layer="91"/>
+<wire x1="-129.54" y1="5.08" x2="-129.54" y2="-2.54" width="0.1524" layer="91"/>
+<junction x="-129.54" y="5.08"/>
+</segment>
+</net>
 </nets>
 </sheet>
@@
 <plain>
 <text x="-96.52" y="43.18" size="1.778" layer="91">POWER SWITCH</text>
-<text x="-91.44" y="5.08" size="1.778" layer="91">5V REG</text>
+<text x="-81.28" y="2.54" size="1.778" layer="91">5V REG</text>
+<text x="15.24" y="17.78" size="1.778" layer="91">POWER OUTPUT</text>
 </plain>
 <instances>
@@
 <attribute name="VALUE" x="-91.44" y="22.86" size="1.778" layer="96"/>
 </instance>
-</instances>
-<busses>
-</busses>
-<nets>
+<instance part="U$7" gate="G$1" x="30.48" y="2.54" smashed="yes">
+<attribute name="NAME" x="20.32" y="13.208" size="1.778" layer="95"/>
+<attribute name="VALUE" x="20.32" y="-2.54" size="1.778" layer="96"/>
+</instance>
+<instance part="X_1" gate="G$1" x="10.16" y="-2.54" smashed="yes"/>
+</instances>
+<busses>
+</busses>
+<nets>
+<net name="24V" class="0">
+<segment>
+<pinref part="U$7" gate="G$1" pin="P$1"/>
+<wire x1="15.24" y1="10.16" x2="0" y2="10.16" width="0.1524" layer="91"/>
+<label x="0" y="10.16" size="1.778" layer="95"/>
+</segment>
+</net>
+<net name="12V" class="0">
+<segment>
+<pinref part="U$7" gate="G$1" pin="P$2"/>
+<wire x1="15.24" y1="7.62" x2="0" y2="7.62" width="0.1524" layer="91"/>
+<label x="0" y="7.62" size="1.778" layer="95"/>
+</segment>
+</net>
+<net name="5V" class="0">
+<segment>
+<pinref part="U$7" gate="G$1" pin="P$3"/>
+<wire x1="15.24" y1="5.08" x2="0" y2="5.08" width="0.1524" layer="91"/>
+<label x="0" y="5.08" size="1.778" layer="95"/>
+</segment>
+</net>
+<net name="0" class="0">
+<segment>
+<pinref part="U$7" gate="G$1" pin="P$4"/>
+<wire x1="15.24" y1="2.54" x2="10.16" y2="2.54" width="0.1524" layer="91"/>
+<wire x1="10.16" y1="2.54" x2="10.16" y2="-2.54" width="0.1524" layer="91"/>
+<pinref part="X_1" gate="G$1" pin="0"/>
+</segment>
+</net>
 </nets>
 </sheet>
@@
 <instances>
 <instance part="U6" gate="G$1" x="0" y="114.3" smashed="yes">
-<attribute name="NAME" x="-15.288" y="162.7117" size="1.783590625" layer="95"/>
-<attribute name="VALUE" x="-15.2708" y="60.8521" size="1.7816" layer="96"/>
+<attribute name="NAME" x="-15.288" y="160.4257" size="1.783590625" layer="95"/>
+<attribute name="VALUE" x="-15.2708" y="63.3921" size="1.7816" layer="96"/>
 </instance>
 <instance part="U7" gate="G$1" x="0" y="-2.54" smashed="yes">
-<attribute name="NAME" x="-15.288" y="45.8717" size="1.783590625" layer="95"/>
-<attribute name="VALUE" x="-15.2708" y="-55.9879" size="1.7816" layer="96"/>
+<attribute name="NAME" x="-15.034" y="43.5857" size="1.783590625" layer="95"/>
+<attribute name="VALUE" x="-15.2708" y="-53.4479" size="1.7816" layer="96"/>
 </instance>
 <instance part="U8" gate="G$1" x="0" y="-111.76" smashed="yes">
-<attribute name="NAME" x="-15.288" y="-63.3483" size="1.783590625" layer="95"/>
-<attribute name="VALUE" x="-15.2708" y="-165.2079" size="1.7816" layer="96"/>
+<attribute name="NAME" x="-15.288" y="-65.6343" size="1.783590625" layer="95"/>
+<attribute name="VALUE" x="-15.2708" y="-162.6679" size="1.7816" layer="96"/>
+</instance>
+<instance part="U$2" gate="G$1" x="106.68" y="116.84" smashed="yes">
+<attribute name="NAME" x="96.52" y="127.508" size="1.778" layer="95"/>
+<attribute name="VALUE" x="96.52" y="111.76" size="1.778" layer="96"/>
+</instance>
+<instance part="U$3" gate="G$1" x="104.14" y="-15.24" smashed="yes">
+<attribute name="NAME" x="93.98" y="-4.572" size="1.778" layer="95"/>
+<attribute name="VALUE" x="93.98" y="-20.32" size="1.778" layer="96"/>
+</instance>
+<instance part="U$4" gate="G$1" x="106.68" y="-121.92" smashed="yes">
+<attribute name="NAME" x="96.52" y="-111.252" size="1.778" layer="95"/>
+<attribute name="VALUE" x="96.52" y="-127" size="1.778" layer="96"/>
 </instance>
 </instances>
@@
 </schematic>
 </drawing>
+<compatibility>
+<note version="8.2" severity="warning">
+Since Version 8.2, EAGLE supports online libraries. The ids
+of those online libraries will not be understood (or retained)
+with this version.
+</note>
+<note version="8.3" severity="warning">
+Since Version 8.3, EAGLE supports URNs for individual library
+assets (packages, symbols, and devices). The URNs of those assets
+will not be understood (or retained) with this version.
+</note>
+</compatibility>
 </eagle>
